Commit message: add moos_gazebo* packages

File: moos_gazebo/config/cora/cora.urdf.xacro (robot description, xacro)
@@ -1,13 +1,13 @@
 <?xml version="1.0"?>
 <robot xmlns:xacro="http://ros.org/wiki/xacro" name="cora">
-  <link name="cora/base_link">
+  <link name="${tf_prefix}/cora/base_link">
   </link>
-  <joint name="cora/dummy_joint" type="fixed">
-    <parent link="cora/base_link"/>
-    <child link="cora/dummy_link"/>
+  <joint name="${tf_prefix}/cora/dummy_joint" type="fixed">
+    <parent link="${tf_prefix}/cora/base_link"/>
+    <child link="${tf_prefix}/cora/dummy_link"/>
     <!-- Adjust the visual/collision to match water height -->
     <origin xyz="0 0 1" rpy="0 0 0"/>
   </joint>
-  <link name="cora/dummy_link">
+  <link name="${tf_prefix}/cora/dummy_link">
     <visual>
       <origin xyz="0 0 0" rpy="0 0 0" />

File: moos_gazebo/config/cora/cora.xacro (robot description, xacro)
@@ -2,18 +2,22 @@
 <robot xmlns:xacro="http://ros.org/wiki/xacro" name="philos">
   <xacro:arg name="locked" default="false" />
+  <xacro:arg name="tf_prefix" default="tf_prefix_not_set"/>
+  <xacro:property name="tf_prefix" value="$(arg tf_prefix)" scope="global"/>
   <!-- Include macros for dynamics plugins -->
-  <xacro:include filename="$(find cora_description)/urdf/macros.xacro" />
+  <xacro:include filename="$(find punch_bringup)/config/cora/macros.xacro" />
   <!-- Attach hydrodynamics plugin -->
   <xacro:usv_dynamics_gazebo name="cora_dynamics_plugin" />
   <!-- Robot mesh -->
-  <xacro:include filename="$(find cora_description)/urdf/cora.urdf.xacro" />
+  <xacro:include filename="$(find punch_bringup)/config/cora/cora.urdf.xacro" />
   <!-- Note: this is only used for some sensors that do not correctly use the
   robotNamespace parameter -->
-  <xacro:arg name="namespace" default="philos"/>
+  <xacro:arg name="namespace" default="namespace_not_set"/>
   <xacro:property name="namespace" value="$(arg namespace)" scope="global" />
   <!-- Thrusters -->
   <xacro:arg name="thruster_namespace" default="thrusters/"/>
   <xacro:property name="thruster_namespace" value="$(arg thruster_namespace)" scope="global" />
-  <xacro:include filename="$(find cora_description)/urdf/thrusters.xacro" />
+  <xacro:arg name="root_namespace" default="root_namespace_not_set"/>
+  <xacro:property name="root_namespace" value="$(arg root_namespace)" scope="global"/>
+  <xacro:include filename="$(find punch_bringup)/config/cora/thrusters.xacro" />
   <!-- Decide if we lock the robot to the world -->
   <xacro:if value="$(arg locked)">
@@ -21,5 +25,5 @@
       <link name="cora_external_link"/>
       <joint name="cora_external_pivot_joint" type="universal">
-        <parent>cora::phios/base_link</parent>
+        <parent>cora::philos/base_link</parent>
         <child>philos_external_link</child>
         <axis>
@@ -49,16 +53,21 @@
   <xacro:property name="camera_namespace" value="$(arg camera_namespace)" scope="global" />
   <xacro:property name="sensor_namespace" value="$(arg sensor_namespace)" scope="global" />
-  <xacro:property name="pinger_namespace" value="$(arg pinger_namespace)" scope="global" />
-  <xacro:wamv_camera name="front_left_camera"  x="-0.61" y="0.2"  z="4.7"
-		     post_z_from="4.6" P="${radians(15)}" Y="${radians(60)}" />
-  <xacro:wamv_camera name="front_center_camera"  x="-0.61" y="0.0"  z="4.7"
-  post_z_from="4.6" P="${radians(15)}" />
-  <xacro:wamv_camera name="front_right_camera" x="-0.61" y="-0.2" z="4.7"
-  post_z_from="4.6" P="${radians(15)}" Y="${radians(-60)}" />
-  <xacro:lidar name="front_lidar" type="16_beam" x="-1.1" z="5"
-  P="${radians(0)}" post_z_from="4.6"/>  <!-- x="-0.595" -->
-  <xacro:wamv_gps name="gps" x="-1.0" z="4.6"
+  <xacro:if value="$(arg sensors)">
+    <xacro:cora_camera name="front_left_camera"  x="-0.61" y="0.2"  z="4.7"
+		       post_z_from="4.6" P="${radians(15)}" Y="${radians(60)}" />
+    <xacro:cora_camera name="front_center_camera"  x="-0.61" y="0.0"  z="4.7"
+		       post_z_from="4.6" P="${radians(15)}" />
+    <xacro:cora_camera name="front_right_camera" x="-0.61" y="-0.2" z="4.7"
+		       post_z_from="4.6" P="${radians(15)}" Y="${radians(-60)}" />
+    <xacro:cora_camera name="side_right_camera" x="-0.75" y="-0.67" z="4.65"
+		       post_z_from="4.55" P="${radians(15)}" Y="${radians(-90)}" />
+    <xacro:lidar name="front_lidar" type="16_beam" x="-1.1" z="5"
+		 P="${radians(0)}" post_z_from="4.6"/>  <!-- x="-0.595" -->
+  </xacro:if>
+  <xacro:cora_gps name="gps" x="-1.0" z="4.6"
   	update_rate="20" />
-  <xacro:wamv_imu name="imu" y="-0.2" z="1.0" update_rate="100" />
-  <xacro:wamv_pinger name="pinger" frameId="cora/pinger" />
+  <xacro:cora_imu name="imu" y="-0.2" z="1.0" update_rate="100" />
+  <xacro:if value="$(arg fiducial)">
+    <xacro:cora_aruco name="aruco" />
+  </xacro:if>
 </robot>

File: moos_gazebo/config/cora/cora_dynamics_plugin.xacro (robot description, xacro)
@@ -5,5 +5,5 @@
     <gazebo>
       <plugin name="usv_dynamics_${name}" filename="libusv_gazebo_dynamics_plugin.so">
-        <bodyName>cora/base_link</bodyName>
+        <bodyName>${tf_prefix}/cora/base_link</bodyName>
         <!-- Must be same as the ocean model!-->
         <waterLevel>0</waterLevel>
@@ -17,7 +17,7 @@
         <nDotR>0.0</nDotR>
         <!-- Linear and quadratic drag -->
-        <xU>120.0</xU>
-        <xUU>240.0</xUU>
-        <yV>240.0</yV>
+        <xU>21200.0</xU>
+        <xUU>22400.0</xUU>
+        <yV>1240.0</yV>
         <yVV>2600</yVV>
         <zW>50000.0</zW>

File: moos_gazebo/config/cora/thrusters.xacro (robot description, xacro)
@@ -2,5 +2,5 @@
 <robot xmlns:xacro="http://ros.org/wiki/xacro">
   <!-- Dummy link, which usv_gazebo_thrust_plugin looks for -->
-  <link name="left_engine_link">
+  <link name="${tf_prefix}/${namespace}/left_engine_link">
     <inertial>
       <mass value="0.1"/>
@@ -9,5 +9,5 @@
   </link>
   <!-- No additional collision, since propeller is inside robot body -->
-  <link name="left_propeller_link">
+  <link name="${tf_prefix}/${namespace}/left_propeller_link">
     <visual>
       <geometry>
@@ -38,21 +38,21 @@
   </link>
   <!-- Dummy joint, which usv_gazebo_thrust_plugin looks for -->
-  <joint name="left_chasis_engine_joint" type="revolute">
+  <joint name="${tf_prefix}/${namespace}/left_chasis_engine_joint" type="revolute">
     <axis xyz="0 0 1"/>
     <origin rpy="0 0 0" xyz="-6.103 0.911 0.016"/>
-    <parent link="cora/base_link"/>
-    <child link="left_engine_link"/>
+    <parent link="${tf_prefix}/${namespace}/base_link"/>
+    <child link="${tf_prefix}/${namespace}/left_engine_link"/>
     <limit lower="${-pi}" upper="${pi}" effort="10" velocity="10"/>
   </joint>
-  <joint name="left_engine_propeller_joint" type="continuous">
+  <joint name="${tf_prefix}/${namespace}/left_engine_propeller_joint" type="continuous">
     <axis rpy="0 0 0" xyz="1 0 0"/>
     <origin xyz="0 0 0" rpy="0 0 0"/>
-    <parent link="left_engine_link"/>
-    <child link="left_propeller_link"/>
+    <parent link="${tf_prefix}/${namespace}/left_engine_link"/>
+    <child link="${tf_prefix}/${namespace}/left_propeller_link"/>
     <limit effort="100" velocity="100" />
     <dynamics friction="0.05" damping="0.05" />
   </joint>
   <!-- Dummy link, which usv_gazebo_thrust_plugin looks for -->
-  <link name="right_engine_link">
+  <link name="${tf_prefix}/${namespace}/right_engine_link">
     <inertial>
       <mass value="0.1"/>
@@ -61,5 +61,5 @@
   </link>
   <!-- No additional collision, since propeller is inside robot body -->
-  <link name="right_propeller_link">
+  <link name="${tf_prefix}/${namespace}/right_propeller_link">
     <visual>
       <geometry>
@@ -90,16 +90,16 @@
   </link>
   <!-- Dummy joint, which usv_gazebo_thrust_plugin looks for -->
-  <joint name="right_chasis_engine_joint" type="revolute">
+  <joint name="${tf_prefix}/${namespace}/right_chasis_engine_joint" type="revolute">
     <axis xyz="0 0 1"/>
     <origin rpy="0 0 0" xyz="-6.103 -0.911 0.016"/>
-    <parent link="cora/base_link"/>
-    <child link="right_engine_link"/>
+    <parent link="${tf_prefix}/${namespace}/base_link"/>
+    <child link="${tf_prefix}/${namespace}/right_engine_link"/>
     <limit lower="${-pi}" upper="${pi}" effort="10" velocity="10"/>
   </joint>
-  <joint name="right_engine_propeller_joint" type="continuous">
+  <joint name="${tf_prefix}/${namespace}/right_engine_propeller_joint" type="continuous">
     <axis rpy="0 0 0" xyz="1 0 0"/>
     <origin xyz="0 0 0" rpy="0 0 0"/>
-    <parent link="right_engine_link"/>
-    <child link="right_propeller_link"/>
+    <parent link="${tf_prefix}/${namespace}/right_engine_link"/>
+    <child link="${tf_prefix}/${namespace}/right_propeller_link"/>
     <limit effort="100" velocity="100" />
     <dynamics friction="0.05" damping="0.05" />
@@ -108,6 +108,6 @@
     <plugin name="cora_gazebo_thrust" filename="libusv_gazebo_thrust_plugin.so">
       <cmdTimeout>1.0</cmdTimeout>
-      <robotNamespace>${namespace}</robotNamespace>
-      <xacro:include filename="$(find cora_description)/urdf/cora_thruster_config.xacro" />
+      <!-- <robotNamespace>${root_namespace}</robotNamespace> -->
+      <xacro:include filename="$(find punch_bringup)/config/cora/cora_thruster_config.xacro" />
       <!-- Angle must be disabled for VORC -->
       <xacro:cora_thruster_config name="left" />
