Commit message: add wamv to sim

File: moos_gazebo/config/cora/macros.xacro (robot description, xacro)
@@ -4,14 +4,13 @@
        name="cora">
   <!-- Include sensor macros -->
-  <xacro:include filename="$(find punch_bringup)/config/cora/cora_camera.xacro" />
-  <!-- Modified for marina world -->
-  <xacro:include filename="$(find punch_bringup)/config/cora/cora_gps.xacro" />
-  <xacro:include filename="$(find punch_bringup)/config/cora/cora_imu.xacro" />
-  <xacro:include filename="$(find punch_bringup)/config/cora/cora_3d_lidar.xacro" />
-  <xacro:include filename="$(find punch_bringup)/config/cora/lidar.xacro" />
-  <xacro:include filename="$(find punch_bringup)/config/cora/cora_p3d.xacro" />
+  <xacro:include filename="$(find moos_gazebo)/config/cora/cora_camera.xacro" />
+  <xacro:include filename="$(find moos_gazebo)/config/cora/cora_gps.xacro" />
+  <xacro:include filename="$(find moos_gazebo)/config/cora/cora_imu.xacro" />
+  <xacro:include filename="$(find moos_gazebo)/config/cora/cora_3d_lidar.xacro" />
+  <xacro:include filename="$(find moos_gazebo)/config/cora/lidar.xacro" />
+  <xacro:include filename="$(find moos_gazebo)/config/cora/cora_p3d.xacro" />
   <!--   -->
-  <xacro:include filename="$(find punch_bringup)/config/cora/cora_aruco.xacro" />
+  <xacro:include filename="$(find moos_gazebo)/config/cora/cora_aruco.xacro" />
   <!-- Include dynamics macros -->
-  <xacro:include filename="$(find punch_bringup)/config/cora/cora_dynamics_plugin.xacro" />
+  <xacro:include filename="$(find moos_gazebo)/config/cora/cora_dynamics_plugin.xacro" />
 </robot>

File: moos_gazebo/config/heron/heron.xacro (robot description, xacro)
@@ -1,13 +1,13 @@
 <?xml version="1.0"?>
-<robot xmlns:xacro="http://ros.org/wiki/xacro" name="cora">
+<robot xmlns:xacro="http://ros.org/wiki/xacro" name="heron">
   <xacro:arg name="locked" default="false" />
   <xacro:arg name="tf_prefix" default="tf_prefix_not_set"/>
   <xacro:property name="tf_prefix" value="$(arg tf_prefix)" scope="global"/>
   <!-- Include macros for dynamics plugins -->
-  <xacro:include filename="$(find moos_gazebo)/config/cora/macros.xacro" />
+  <xacro:include filename="$(find moos_gazebo)/config/heron/macros.xacro" />
   <!-- Attach hydrodynamics plugin -->
-  <xacro:usv_dynamics_gazebo name="cora_dynamics_plugin" />
-  <!-- Robot mesh -->
-  <xacro:include filename="$(find moos_gazebo)/config/cora/cora.urdf.xacro" />
+  <xacro:usv_dynamics_gazebo name="heron_dynamics_plugin" />
+  <!-- Robot mesh   -->
+  <xacro:include filename="$(find moos_gazebo)/config/heron/heron.urdf.xacro" />
   <!-- Note: this is only used for some sensors that do not correctly use the
   robotNamespace parameter -->
@@ -19,12 +19,12 @@
   <xacro:arg name="root_namespace" default="root_namespace_not_set"/>
   <xacro:property name="root_namespace" value="$(arg root_namespace)" scope="global"/>
-  <xacro:include filename="$(find moos_gazebo)/config/cora/thrusters.xacro" />
+  <xacro:include filename="$(find moos_gazebo)/config/heron/thrusters.xacro" />
   <!-- Decide if we lock the robot to the world -->
   <xacro:if value="$(arg locked)">
     <gazebo>
-      <link name="cora_external_link"/>
-      <joint name="cora_external_pivot_joint" type="universal">
-        <parent>cora::cora/base_link</parent>
-        <child>cora_external_link</child>
+      <link name="heron_external_link"/>
+      <joint name="heron_external_pivot_joint" type="universal">
+        <parent>heron::heron/base_link</parent>
+        <child>heron_external_link</child>
         <axis>
           <xyz>1 0 0</xyz>
@@ -34,7 +34,7 @@
         </axis2>
       </joint>
-      <joint name="cora_external_riser" type="prismatic">
+      <joint name="heron_external_riser" type="prismatic">
         <parent>world</parent>
-        <child>cora_external_link</child>
+        <child>heron_external_link</child>
         <axis>
           <limit>
@@ -53,21 +53,23 @@
   <xacro:property name="camera_namespace" value="$(arg camera_namespace)" scope="global" />
   <xacro:property name="sensor_namespace" value="$(arg sensor_namespace)" scope="global" />
+  <!--
   <xacro:if value="$(arg sensors)">
-    <xacro:cora_camera name="front_left_camera"  x="-0.61" y="0.2"  z="4.7"
+    <xacro:heron_camera name="front_left_camera"  x="-0.61" y="0.2"  z="4.7"
 		       post_z_from="4.6" P="${radians(15)}" Y="${radians(60)}" />
-    <xacro:cora_camera name="front_center_camera"  x="-0.61" y="0.0"  z="4.7"
+    <xacro:heron_camera name="front_center_camera"  x="-0.61" y="0.0"  z="4.7"
 		       post_z_from="4.6" P="${radians(15)}" />
-    <xacro:cora_camera name="front_right_camera" x="-0.61" y="-0.2" z="4.7"
+    <xacro:heron_camera name="front_right_camera" x="-0.61" y="-0.2" z="4.7"
 		       post_z_from="4.6" P="${radians(15)}" Y="${radians(-60)}" />
-    <xacro:cora_camera name="side_right_camera" x="-0.75" y="-0.67" z="4.65"
+    <xacro:heron_camera name="side_right_camera" x="-0.75" y="-0.67" z="4.65"
 		       post_z_from="4.55" P="${radians(15)}" Y="${radians(-90)}" />
     <xacro:lidar name="front_lidar" type="16_beam" x="-1.1" z="5"
-		 P="${radians(0)}" post_z_from="4.6"/>  <!-- x="-0.595" -->
+		 P="${radians(0)}" post_z_from="4.6"/>
   </xacro:if>
-  <xacro:cora_gps name="gps" x="-1.0" z="4.6"
+  <xacro:heron_gps name="gps" x="-1.0" z="4.6"
   	update_rate="20" />
-  <xacro:cora_imu name="imu" y="-0.2" z="1.0" update_rate="100" />
+  <xacro:heron_imu name="imu" y="-0.2" z="1.0" update_rate="100" />
+  -->
   <xacro:if value="$(arg fiducial)">
-    <xacro:cora_aruco name="aruco" />
+    <xacro:heron_aruco name="aruco" />
   </xacro:if>
 </robot>

File: moos_gazebo/config/heron/lidar.xacro (robot description, xacro)
@@ -1,5 +1,5 @@
 <?xml version="1.0" encoding="UTF-8"?>
 <robot xmlns:xacro="http://ros.org/wiki/xacro">
-  <xacro:include filename="$(find moos_gazebo)/config/cora/cora_3d_lidar.xacro"/>
+  <xacro:include filename="$(find moos_gazebo)/config/heron/heron_3d_lidar.xacro"/>
   <xacro:macro name="lidar"
                params = "type:='16_beam'

File: moos_gazebo/config/heron/thrusters.xacro (robot description, xacro)
@@ -12,5 +12,5 @@
     <visual>
       <geometry>
-        <mesh filename="package://cora_description/models/meshes/propellerL.dae"/>
+        <mesh filename="package://heron_description/models/meshes/propellerL.dae"/>
       </geometry>
       <material name="left_propeller_material">
@@ -19,13 +19,13 @@
         <pbr>
           <metal>
-            <albedo_map>package://cora_description/models/materials/textures/Boat_Albedo.png</albedo_map>
-            <metalness_map>package://cora_description/models/materials/textures/Boat_Metalness.png</metalness_map>
-            <roughness_map>package://cora_description/models/materials/textures/Boat_Roughness.png</roughness_map>
+            <albedo_map>package://heron_description/models/materials/textures/Boat_Albedo.png</albedo_map>
+            <metalness_map>package://heron_description/models/materials/textures/Boat_Metalness.png</metalness_map>
+            <roughness_map>package://heron_description/models/materials/textures/Boat_Roughness.png</roughness_map>
           </metal>
         </pbr>
         <!-- fallback to script if no PBR support-->
         <script>
-          <uri>package://cora_description/models/materials/scripts/</uri>
-          <uri>package://cora_description/models/materials/textures/</uri>
+          <uri>package://heron_description/models/materials/scripts/</uri>
+          <uri>package://heron_description/models/materials/textures/</uri>
           <name>UrbanTile/Boat_Diffuse</name>
         </script>
@@ -64,5 +64,5 @@
     <visual>
       <geometry>
-        <mesh filename="package://cora_description/models/meshes/propellerR.dae"/>
+        <mesh filename="package://heron_description/models/meshes/propellerR.dae"/>
       </geometry>
       <material name="right_propeller_material">
@@ -71,13 +71,13 @@
         <pbr>
           <metal>
-            <albedo_map>package://cora_description/models/materials/textures/Boat_Albedo.png</albedo_map>
-            <metalness_map>package://cora_description/models/materials/textures/Boat_Metalness.png</metalness_map>
-            <roughness_map>package://cora_description/models/materials/textures/Boat_Roughness.png</roughness_map>
+            <albedo_map>package://heron_description/models/materials/textures/Boat_Albedo.png</albedo_map>
+            <metalness_map>package://heron_description/models/materials/textures/Boat_Metalness.png</metalness_map>
+            <roughness_map>package://heron_description/models/materials/textures/Boat_Roughness.png</roughness_map>
           </metal>
         </pbr>
         <!-- fallback to script if no PBR support-->
         <script>
-          <uri>package://cora_description/models/materials/scripts/</uri>
-          <uri>package://cora_description/models/materials/textures/</uri>
+          <uri>package://heron_description/models/materials/scripts/</uri>
+          <uri>package://heron_description/models/materials/textures/</uri>
           <name>UrbanTile/Boat_Diffuse</name>
         </script>
@@ -106,11 +106,11 @@
   </joint>
   <gazebo>
-    <plugin name="cora_gazebo_thrust" filename="libusv_gazebo_thrust_plugin.so">
+    <plugin name="heron_gazebo_thrust" filename="libusv_gazebo_thrust_plugin.so">
       <cmdTimeout>1.0</cmdTimeout>
       <!-- <robotNamespace>${root_namespace}</robotNamespace> -->
-      <xacro:include filename="$(find moos_gazebo)/config/cora/cora_thruster_config.xacro" />
+      <xacro:include filename="$(find moos_gazebo)/config/heron/heron_thruster_config.xacro" />
       <!-- Angle must be disabled for VORC -->
-      <xacro:cora_thruster_config name="left" />
-      <xacro:cora_thruster_config name="right" />
+      <xacro:heron_thruster_config name="left" />
+      <xacro:heron_thruster_config name="right" />
     </plugin>
   </gazebo>
