Commit message: test and update launch files

File: moos_gazebo/config/cora/cora.xacro (robot description, xacro)
@@ -1,13 +1,13 @@
 <?xml version="1.0"?>
-<robot xmlns:xacro="http://ros.org/wiki/xacro" name="philos">
+<robot xmlns:xacro="http://ros.org/wiki/xacro" name="cora">
   <xacro:arg name="locked" default="false" />
   <xacro:arg name="tf_prefix" default="tf_prefix_not_set"/>
   <xacro:property name="tf_prefix" value="$(arg tf_prefix)" scope="global"/>
-  <!-- Include macros for dynamic plugins -->
-  <xacro:include filename="$(find punch_bringup)/config/cora/macros.xacro" />
+  <!-- Include macros for dynamics plugins -->
+  <xacro:include filename="$(find moos_gazebo)/config/cora/macros.xacro" />
   <!-- Attach hydrodynamics plugin -->
   <xacro:usv_dynamics_gazebo name="cora_dynamics_plugin" />
   <!-- Robot mesh -->
-  <xacro:include filename="$(find punch_bringup)/config/cora/cora.urdf.xacro" />
+  <xacro:include filename="$(find moos_gazebo)/config/cora/cora.urdf.xacro" />
   <!-- Note: this is only used for some sensors that do not correctly use the
   robotNamespace parameter -->
@@ -19,5 +19,5 @@
   <xacro:arg name="root_namespace" default="root_namespace_not_set"/>
   <xacro:property name="root_namespace" value="$(arg root_namespace)" scope="global"/>
-  <xacro:include filename="$(find punch_bringup)/config/cora/thrusters.xacro" />
+  <xacro:include filename="$(find moos_gazebo)/config/cora/thrusters.xacro" />
   <!-- Decide if we lock the robot to the world -->
   <xacro:if value="$(arg locked)">
@@ -25,6 +25,6 @@
       <link name="cora_external_link"/>
       <joint name="cora_external_pivot_joint" type="universal">
-        <parent>cora::philos/base_link</parent>
-        <child>philos_external_link</child>
+        <parent>cora::cora/base_link</parent>
+        <child>cora_external_link</child>
         <axis>
           <xyz>1 0 0</xyz>
@@ -36,5 +36,5 @@
       <joint name="cora_external_riser" type="prismatic">
         <parent>world</parent>
-        <child>philos_external_link</child>
+        <child>cora_external_link</child>
         <axis>
           <limit>

File: moos_gazebo/config/cora/lidar.xacro (robot description, xacro)
@@ -1,5 +1,5 @@
 <?xml version="1.0" encoding="UTF-8"?>
 <robot xmlns:xacro="http://ros.org/wiki/xacro">
-  <xacro:include filename="$(find punch_bringup)/config/cora/cora_3d_lidar.xacro"/>
+  <xacro:include filename="$(find moos_gazebo)/config/cora/cora_3d_lidar.xacro"/>
   <xacro:macro name="lidar"
                params = "type:='16_beam'

File: moos_gazebo/config/cora/thrusters.xacro (robot description, xacro)
@@ -109,5 +109,5 @@
       <cmdTimeout>1.0</cmdTimeout>
       <!-- <robotNamespace>${root_namespace}</robotNamespace> -->
-      <xacro:include filename="$(find punch_bringup)/config/cora/cora_thruster_config.xacro" />
+      <xacro:include filename="$(find moos_gazebo)/config/cora/cora_thruster_config.xacro" />
       <!-- Angle must be disabled for VORC -->
       <xacro:cora_thruster_config name="left" />

Commit message: add aruco to port and starboard of cora, add macros to cora_aruco

File: moos_gazebo/config/cora/cora.xacro (robot description, xacro)
@@ -69,5 +69,6 @@
   <xacro:cora_imu name="imu" y="-0.2" z="1.0" update_rate="100" />
   <xacro:if value="$(arg fiducial)">
-    <xacro:cora_aruco name="aruco" />
+    <xacro:cora_aruco name="starboard_aruco" x="-1.0" y="1.0" z="4.0" R="0" P="0" Y="1.57"  />
+    <xacro:cora_aruco name="port_aruco" x="-1.0" y="-1.0" z="4.0" R="0" P="0" Y="1.57"  />
   </xacro:if>
 </robot>

File: moos_gazebo/config/cora/cora_aruco.xacro (robot description, xacro)
@@ -36,10 +36,10 @@
       </inertial>
     </link>
-    <joint name="aruco_joint" type="fixed">
+    <joint name="${name}_joint" type="fixed">
       <parent link="${tf_prefix}/${namespace}/base_link"/>
       <child link="${tf_prefix}/${namespace}/${name}_link"/>
-      <origin xyz="-1.0 1.0 4.0" rpy="0 0 1.57"/>
+      <origin xyz="${x} ${y} ${z}" rpy="${R} ${P} ${Y}"/>
     </joint>
-    <link name="aruco_marker">
+    <link name="${name}_marker">
       <collision>
 	<origin xyz="0 0 0" rpy="0 0 0"/>
@@ -55,10 +55,11 @@
       </visual>
     </link>
-    <joint name="aruco_marker_link" type="fixed">
+    <joint name="${name}_marker_link" type="fixed">
       <parent link="${tf_prefix}/${namespace}/base_link"/>
-      <child  link="aruco_marker"/>
-      <origin xyz="-1.0 1.01 4.0" rpy="0 0 1.57"/>
+      <child  link="${name}_marker"/>
+      <origin xyz="${x} ${y}1 ${z}" rpy="${R} ${P} ${Y}"/>
+      <!-- add 1 to end of y to place marker on top of board -->
     </joint>
-    <gazebo reference="aruco_marker">
+    <gazebo reference="${name}_marker">
       <material>aruco_26</material>
     </gazebo>

File: moos_gazebo/config/wamv/wamv.xacro (robot description, xacro)
@@ -10,5 +10,5 @@
   <xacro:property name="namespace" value="$(arg namespace)" scope="global"/>
   <!-- Robot Mesh -->
-  <xacro:include filename="$(find moos_gazebo)/config/wamv/wamv_base.urdf.xacro"/> -->
+  <xacro:include filename="$(find moos_gazebo)/config/wamv/wamv_base.urdf.xacro"/>
   <!-- Load Sensors -->
   <xacro:arg name="sensor_namespace" default="sensors/"/>
