Commit message: update namespacing for thrusters and base urdf model

File: moos_gazebo/config/wamv/wamv.xacro (robot description, xacro)
@@ -1,9 +1,11 @@
 <?xml version="1.0" ?>
-<robot xmlns:xacro="http://ros.org/wiki/xacro" name="rex4">
-  <!-- Robot Mesh -->
-  <xacro:include filename="$(find moos_gazebo)/config/wamv/wamv_base.urdf.xacro"/> -->
+<robot xmlns:xacro="http://ros.org/wiki/xacro" name="wamv">
+  <xacro:arg name="tf_prefix" default="tf_prefix_not_set"/>
+  <xacro:property name="tf_prefix" value="$(arg tf_prefix)" scope="global"/>
   <!-- Note: this is only used for some sensors that do not correctly use
        the robotNamespace parameter -->
   <xacro:arg name="namespace" default="namespace_not_set"/>
   <xacro:property name="namespace" value="$(arg namespace)" scope="global"/>
+  <!-- Robot Mesh -->
+  <xacro:include filename="$(find moos_gazebo)/config/wamv/wamv_base_2.urdf.xacro"/> -->
 </robot>

Commit message: adding components to wamv config, fixing namespacing macros

File: moos_gazebo/config/wamv/wamv.xacro (robot description, xacro)
@@ -1,4 +1,6 @@
 <?xml version="1.0" ?>
 <robot xmlns:xacro="http://ros.org/wiki/xacro" name="wamv">
+  <!-- Include macros for dynamic plugins -->
+  <xacro:include filename="$(find moos_gazebo)/config/wamv/components/component_macros.xacro" />
   <xacro:arg name="tf_prefix" default="tf_prefix_not_set"/>
   <xacro:property name="tf_prefix" value="$(arg tf_prefix)" scope="global"/>
@@ -9,3 +11,22 @@
   <!-- Robot Mesh -->
   <xacro:include filename="$(find moos_gazebo)/config/wamv/wamv_base.urdf.xacro"/> -->
+  <!-- Load Sensors -->
+  <xacro:arg name="sensor_namespace" default="sensors/"/>
+  <xacro:property name="sensor_namespace" value="$(arg sensor_namespace)" scope="global"/>
+  <xacro:arg name="camera_namespace" default="cameras/"/>
+  <xacro:property name="camera_namespace" value="$(arg camera_namespace)" scope="global"/>
+  <!-- Front Camera Generic if there is not a URDF set up by camera driver: 'camera.xacro' -->
+  <xacro:camera name="front_camera" x="0.75" y="0.0" z="1.7283" />
+  <!-- OAK-D TF and URDF is launch within the specific launch file -->
+  <!-- Port Camera Generic: 'camera.xacro' -->
+  <!-- Front Lidar -->
+  <xacro:lidar name="front_lidar" x="0.75" z="1.7828"/>
+  <!-- IMU/GNSS  -->
+  <xacro:imu name="imu_gnss_xsens" x="0.77" />
+  <!-- GPS -->
+  <xacro:gps name="gps_hemisphere" x="-0.75"  />
+  <!-- Marine Radar -->
+  <!-- This is only a model to represent transforms,
+       do not yet have a working marine radar simulator -->
+  <xacro:radar name="radar_broadband" x="0.75" z="1.95"/>
 </robot>
