Commit message: updates

File: moos_gazebo/config/wamv/components/camera.xacro (robot description, xacro)
@@ -127,4 +127,51 @@
       <child link="${tf_prefix}/${namespace}/${name}_link_optical" />
     </joint>
+    <!-- Gazebo camera setup -->
+    <gazebo reference="${tf_prefix}/${namespace}/${name}_link">
+      <sensor type="camera" name="${name}_sensor">
+        <update_rate>30.0</update_rate>
+        <xacro:if value="${visualize}">
+          <visualize>true</visualize>
+        </xacro:if>
+        <camera name="${name}_camera">
+          <horizontal_fov>1.3962634</horizontal_fov>
+          <image>
+            <width>1280</width>
+            <height>720</height>
+            <format>R8G8B8</format>
+          </image>
+          <clip>
+            <near>0.05</near>
+            <far>300</far>
+          </clip>
+          <noise>
+            <type>gaussian</type>
+            <!-- Noise is sampled independently per pixel on each frame.
+                 That pixel's noise value is added to each of its color
+                 channels, which at that point lie in the range [0,1]. -->
+            <mean>0.0</mean>
+            <stddev>0.007</stddev>
+          </noise>
+        </camera>
+        <plugin name="camera_plugin_${name}" filename="libgazebo_ros_camera.so">
+          <alwaysOn>true</alwaysOn>
+          <updateRate>0.0</updateRate>
+          <cameraName>${namespace}/${sensor_namespace}${camera_namespace}${name}</cameraName>
+          <imageTopicName>image_raw</imageTopicName>
+          <cameraInfoTopicName>camera_info</cameraInfoTopicName>
+          <frameName>${tf_prefix}/${namespace}/${name}_link_optical</frameName>
+          <hackBaseline>0.07</hackBaseline>
+          <distortionK1>0.0</distortionK1>
+          <distortionK2>0.0</distortionK2>
+          <distortionK3>0.0</distortionK3>
+          <distortionT1>0.0</distortionT1>
+          <distortionT2>0.0</distortionT2>
+        </plugin>
+      </sensor>
+    </gazebo>
+    <!-- Set color of post -->
+    <gazebo reference="${tf_prefix}/${namespace}/${name}_post_link">
+      <material>Gazebo/Black</material>
+    </gazebo>
   </xacro:macro>
 </robot>
