Commit message: general cleanup

File: moos_gazebo/config/wamv/components/imu.xacro (robot description, xacro)
@@ -3,5 +3,5 @@
   <xacro:macro name="imu" params="name:=imu x:=0.3 y:=0.0 z:=1.3 R:=0 P:=0 Y:=0 update_rate:=15">
     <link name="${tf_prefix}/${namespace}/${name}_link">
-      <visual name="${name}_visual">>
+      <visual name="${name}_visual">
         <geometry>
           <box size="0.05 0.025 0.005" />

File: moos_gazebo/config/wamv/wamv_base.urdf.xacro (robot description, xacro)
@@ -2,5 +2,5 @@
 <!-- WAMV Base with namespace changes 2023-12-12 -->
 <!-- Basic WAM-V with gazebo plugins for dynamics -->
-<robot name="WAM-V">
+<robot name="wamv">
   <link name="${tf_prefix}/${namespace}/left_battery_link">
     <visual name="left_battery_visual">
